Commit message: add 2x versions of artags

File: urdf/artag_2x.urdf.xacro (robot description, xacro)
@@ -16,5 +16,5 @@
         <origin xyz="0 0 0" rpy="0 -1.57079632679 0"/>
         <geometry>
-          <mesh filename="package://vigir_ar_alvar_description/meshes/${name}.dae"/>
+          <mesh filename="package://vigir_ar_alvar_description/meshes/${name}_2x.dae"/>
         </geometry>
       </visual>
@@ -22,5 +22,5 @@
         <origin xyz="0 0 0" rpy="0 0 0"/>
         <geometry>
-          <mesh filename="package://vigir_ar_alvar_description/meshes/${name}.dae"/>
+          <mesh filename="package://vigir_ar_alvar_description/meshes/${name}_2x.dae"/>
         </geometry>
       </collision>
@@ -40,5 +40,5 @@
         <origin xyz="0 0 0" rpy="0 0 0"/>
         <geometry>
-          <box size="0.1 0.1 0.001" />
+          <box size="0.2 0.2 0.001" />
         </geometry>
       </visual>
@@ -46,5 +46,5 @@
         <origin xyz="0 0 0" rpy="0 0 0"/>
         <geometry>
-          <box size="0.1 0.1 0.0001" />
+          <box size="0.2 0.2 0.0001" />
         </geometry>
       </collision>
